Commit message: 26.12.19

File: dql_robot/urdf/object_disposer_robot/hokuyo.xacro (robot description, xacro)
@@ -43,5 +43,5 @@
             <range>
               <min>0.08</min>
-              <max>5</max>
+              <max>50</max>
               <resolution>0.01</resolution>
             </range>
@@ -49,5 +49,5 @@
           <plugin name="laser" filename="libgazebo_ros_laser.so" >
               <!--<robotNamespace></robotNamespace>-->
-            <topicName>scan</topicName>
+            <topicName>laser_scans</topicName>
             <frameName>base_laser</frameName>
           </plugin>

File: dql_robot/urdf/object_disposer_robot/my_robot_a.SLDASM.urdf.xacro (robot description, xacro)
@@ -639,7 +639,72 @@
     </sensor>
   </gazebo>
+   <joint name="hokuyo_joint" type="fixed">
+    <axis xyz="0 1 0" />
+    <origin xyz="-1.1 0 0.20" rpy="0 0 3.1415"/>
+    <parent link="base_link"/>
+    <child link="hokuyo_link"/>
+  </joint>
+  <!-- Hokuyo Laser -->
+  <link name="hokuyo_link">
+    <collision>
+      <origin xyz="0 0 0" rpy="0 0 0"/>
+      <geometry>
+    <box size="0.1 0.1 0.1"/>
+      </geometry>
+    </collision>
+    <visual>
+      <origin xyz="0 0 0" rpy="0 0 0"/>
+      <geometry>
+        <mesh filename="package://dql_robot/urdf/hokuyo.dae"/>
+      </geometry>
+    </visual>
+    <inertial>
+      <mass value="1e-5" />
+      <origin xyz="0 0 0" rpy="0 0 0"/>
+      <inertia ixx="1e-6" ixy="0" ixz="0" iyy="1e-6" iyz="0" izz="1e-6" />
+    </inertial>
+  </link>
+<gazebo reference="hokuyo_link">
+   <!-- <sensor type="gpu_ray" name="head_hokuyo_sensor">-->
+   <sensor type="ray" name="head_hokuyo_sensor">
+      <pose>0 0 0 0 0 0</pose>
+      <visualize>true</visualize>
+      <update_rate>100</update_rate>
+      <ray>
+        <scan>
+          <horizontal>
+            <samples>720</samples>
+            <resolution>1</resolution>
+            <min_angle>-1.570796</min_angle>
+            <max_angle>1.570796</max_angle>
+          </horizontal>
+        </scan>
+        <range>
+          <min>0.1</min>
+          <max>50.0</max>
+          <resolution>0.1</resolution>
+        </range>
+        <noise>
+          <type>gaussian</type>
+          <!-- Noise parameters based on published spec for Hokuyo laser
+               achieving "+-30mm" accuracy at range < 10m.  A mean of 0.0m and
+               stddev of 0.01m will put 99.7% of samples within 0.03m of the true
+               reading. -->
+          <mean>0.0</mean>
+          <stddev>0.01</stddev>
+        </noise>
+      </ray>
+     <!-- <plugin name="gazebo_ros_head_hokuyo_controller" filename="libgazebo_ros_gpu_laser.so">-->
+     <plugin name="gazebo_ros_head_hokuyo_controller" filename="libgazebo_ros_laser.so">
+        <topicName>scan</topicName>
+        <frameName>hokuyo_link</frameName>
+      </plugin>
+    </sensor>
+  </gazebo>
 <!-- camera-->
 <xacro:property name="camera_link1" value="0.05" /> <!-- Size of square 'camera' box -->
 <xacro:property name="camera_link2" value="0.05" /> <!-- Size of square 'camera' box -->
+<!--laser-->
+<xacro:property name="hokuyo_link" value="0.05" />
 <!-- lazer scanner -->
 <!--
