Commit message: 12.04.20

File: dql_robot/urdf/object_disposer_robot/my_robot_a.SLDASM.urdf (backup).xacro (robot description, xacro)
@@ -77,10 +77,9 @@
     <collision>
       <origin
-        xyz="0 0 0"
-        rpy="0 0 0" />
-      <geometry>
-        <mesh
-          filename="package://dql_robot/meshes_object_disposer_robot/left_front.STL" />
-      </geometry>
+        xyz="0 0 0.13"
+        rpy="0 pi 0" />
+      <geometry>
+    <cylinder length="0.1" radius="0.25"/>
+    </geometry>
     </collision>
   </link>
@@ -98,6 +97,5 @@
       xyz="0 1 0" />
   </joint>
-  <link
-    name="left_front_r">
+  <link name="left_front_r">
     <inertial>
       <origin
@@ -130,10 +128,9 @@
     <collision>
       <origin
-        xyz="0 0 0"
-        rpy="0 0 0" />
-      <geometry>
-        <mesh
-          filename="package://dql_robot/meshes_object_disposer_robot/left_front_r.STL" />
-      </geometry>
+        xyz="0 0 0.13"
+        rpy="0 0 0" />
+      <geometry>
+    <cylinder length="0.1" radius="0.25"/>
+    </geometry>
     </collision>
   </link>
@@ -183,10 +180,9 @@
     <collision>
       <origin
-        xyz="0 0 0"
-        rpy="0 0 0" />
-      <geometry>
-        <mesh
-          filename="package://dql_robot/meshes_object_disposer_robot/left_back.STL" />
-      </geometry>
+        xyz="0 0 0.13"
+        rpy="0 pi 0" />
+      <geometry>
+        <cylinder length="0.1" radius="0.25"/>
+    </geometry>
     </collision>
   </link>
@@ -236,10 +232,9 @@
     <collision>
       <origin
-        xyz="0 0 0"
-        rpy="0 0 0" />
-      <geometry>
-        <mesh
-          filename="package://dql_robot/meshes_object_disposer_robot/left_back_r.STL" />
-      </geometry>
+        xyz="0 0 0.13"
+        rpy="0 0 0" />
+      <geometry>
+    <cylinder length="0.1" radius="0.25"/>
+    </geometry>
     </collision>
   </link>
@@ -289,10 +284,9 @@
     <collision>
       <origin
-        xyz="0 0 0"
-        rpy="0 0 0" />
-      <geometry>
-        <mesh
-          filename="package://dql_robot/meshes_object_disposer_robot/right_front.STL" />
-      </geometry>
+        xyz="0 0 0.13"
+        rpy="0 pi 0" />
+      <geometry>
+        <cylinder length="0.1" radius="0.25"/>
+    </geometry>
     </collision>
   </link>
@@ -342,10 +336,9 @@
     <collision>
       <origin
-        xyz="0 0 0"
-        rpy="0 0 0" />
-      <geometry>
-        <mesh
-          filename="package://dql_robot/meshes_object_disposer_robot/right_front_r.STL" />
-      </geometry>
+        xyz="0 0 -0.13"
+        rpy="0 0 0" />
+      <geometry>
+    <cylinder length="0.1" radius="0.25"/>
+    </geometry>
     </collision>
   </link>
@@ -395,10 +388,9 @@
     <collision>
       <origin
-        xyz="0 0 0"
-        rpy="0 0 0" />
-      <geometry>
-        <mesh
-          filename="package://dql_robot/meshes_object_disposer_robot/right_back.STL" />
-      </geometry>
+        xyz="0 0 -0.13"
+        rpy="0 pi 0" />
+      <geometry>
+        <cylinder length="0.1" radius="0.25"/>
+    </geometry>
     </collision>
   </link>
@@ -448,10 +440,9 @@
     <collision>
       <origin
-        xyz="0 0 0"
-        rpy="0 0 0" />
-      <geometry>
-        <mesh
-          filename="package://dql_robot/meshes_object_disposer_robot/right_back_r.STL" />
-      </geometry>
+        xyz="0 -0.011 -0.13"
+        rpy="0 0 0" />
+      <geometry>
+    <cylinder length="0.1" radius="0.25"/>
+    </geometry>
     </collision>
   </link>
@@ -576,5 +567,5 @@
   <joint name="camera_joint2" type="fixed">
     <axis xyz="0 -1 0" />
-    <origin xyz="-10.0 0.0 10.0" rpy="0 1.545 3.14"/> <!--z=12-->
+    <origin xyz="-10.0 0.0 12.0" rpy="0 1.545 3.14"/>
     <parent link="base_link"/>
     <child link="camera_link2"/>
