Commit message: update added video recorder and new reset ruls

File: dql_robot/urdf/object_disposer_robot/my_robot_a.SLDASM.urdf.xacro (robot description, xacro)
@@ -539,5 +539,5 @@
   <joint name="camera_joint1" type="fixed">
     <axis xyz="0 -1 0" />
-    <origin xyz="-0.8 0.0 0.8" rpy="0 0 600"/>
+    <origin xyz="-0.8 0.0 1.0" rpy="0 0.45 3.14"/>
     <parent link="base_link"/>
     <child link="camera_link1"/>

Commit message: update

File: dql_robot/urdf/object_disposer_robot/my_robot_a.SLDASM.urdf.xacro (robot description, xacro)
@@ -542,4 +542,30 @@
     <parent link="base_link"/>
     <child link="camera_link1"/>
+  </joint>
+<link name="camera_link2">
+    <collision>
+      <origin xyz="0 0 0" rpy="0 0 0"/>
+      <geometry>
+    <box size="0.1 0.1 0.1"/>
+      </geometry>
+    </collision>
+    <visual>
+      <origin xyz="0 0 0" rpy="0 0 0"/>
+      <geometry>
+    <box size="0.1 0.1 0.1"/>
+      </geometry>
+      <material name="red"/>
+    </visual>
+    <inertial>
+      <mass value="1e-5" />
+      <origin xyz="0 0 0" rpy="0 0 0"/>
+      <inertia ixx="1e-6" ixy="0" ixz="0" iyy="1e-6" iyz="0" izz="1e-6" />
+    </inertial>
+  </link>
+  <joint name="camera_joint2" type="fixed">
+    <axis xyz="0 -1 0" />
+    <origin xyz="-20.0 0.0 12.0" rpy="0 1.545 3.14"/>
+    <parent link="base_link"/>
+    <child link="camera_link2"/>
   </joint>
  <gazebo reference="camera_link1">
@@ -582,6 +608,46 @@
     </sensor>
   </gazebo>
+   <gazebo reference="camera_link2">
+    <sensor type="camera" name="camera2">
+      <update_rate>30.0</update_rate>
+      <camera name="head">
+        <horizontal_fov>2.5</horizontal_fov>
+        <image>
+          <width>640</width>
+          <height>480</height>
+          <format>R8G8B8</format>
+        </image>
+        <clip>
+          <near>0.15</near>
+          <far>300</far>
+        </clip>
+        <noise>
+          <type>gaussian</type>
+          <!-- Noise is sampled independently per pixel on each frame.
+               That pixel's noise value is added to each of its color
+               channels, which at that point lie in the range [0,1]. -->
+          <mean>0.0</mean>
+          <stddev>0.007</stddev>
+        </noise>
+      </camera>
+      <plugin name="camera_controller" filename="libgazebo_ros_camera.so">
+        <alwaysOn>true</alwaysOn>
+        <updateRate>0.0</updateRate>
+        <cameraName>/top_camera</cameraName>
+        <imageTopicName>image_raw</imageTopicName>
+        <cameraInfoTopicName>camera_info</cameraInfoTopicName>
+        <frameName>camera_link1</frameName>
+        <hackBaseline>0.07</hackBaseline>
+        <distortionK1>0.0</distortionK1>
+        <distortionK2>0.0</distortionK2>
+        <distortionK3>0.0</distortionK3>
+        <distortionT1>0.0</distortionT1>
+        <distortionT2>0.0</distortionT2>
+      </plugin>
+    </sensor>
+  </gazebo>
 <!-- camera-->
 <xacro:property name="camera_link1" value="0.05" /> <!-- Size of square 'camera' box -->
+<xacro:property name="camera_link2" value="0.05" /> <!-- Size of square 'camera' box -->
 <!-- lazer scanner -->
 <!--

Commit message: las

File: dql_robot/urdf/object_disposer_robot/my_robot_a.SLDASM.urdf.xacro (robot description, xacro)
@@ -132,8 +132,7 @@
         xyz="0 0 0"
         rpy="0 0 0" />
-      <geometry>
-        <mesh
-          filename="package://dql_robot/meshes_object_disposer_robot/left_front_r.STL" />
-      </geometry>
+<geometry>
+    <cylinder length="0.3" radius="0.3"/>
+</geometry>
     </collision>
   </link>

Commit message: galil

File: dql_robot/urdf/object_disposer_robot/my_robot_a.SLDASM.urdf.xacro (robot description, xacro)
@@ -77,10 +77,9 @@
     <collision>
       <origin
-        xyz="0 0 0"
-        rpy="0 0 0" />
-      <geometry>
-        <mesh
-          filename="package://dql_robot/meshes_object_disposer_robot/left_front.STL" />
-      </geometry>
+        xyz="0 0 0.13"
+        rpy="0 pi 0" />
+      <geometry>
+    <cylinder length="0.3" radius="0.12"/>
+    </geometry>
     </collision>
   </link>
@@ -130,9 +129,9 @@
     <collision>
       <origin
-        xyz="0 0 0"
-        rpy="0 0 0" />
-<geometry>
-    <cylinder length="0.3" radius="0.3"/>
-</geometry>
+        xyz="0 0 0.13"
+        rpy="0 0 0" />
+      <geometry>
+    <cylinder length="0.3" radius="0.25"/>
+    </geometry>
     </collision>
   </link>
@@ -182,10 +181,9 @@
     <collision>
       <origin
-        xyz="0 0 0"
-        rpy="0 0 0" />
-      <geometry>
-        <mesh
-          filename="package://dql_robot/meshes_object_disposer_robot/left_back.STL" />
-      </geometry>
+        xyz="0 0 0.13"
+        rpy="0 pi 0" />
+      <geometry>
+    <cylinder length="0.3" radius="0.12"/>
+    </geometry>
     </collision>
   </link>
@@ -235,10 +233,9 @@
     <collision>
       <origin
-        xyz="0 0 0"
-        rpy="0 0 0" />
-      <geometry>
-        <mesh
-          filename="package://dql_robot/meshes_object_disposer_robot/left_back_r.STL" />
-      </geometry>
+        xyz="0 0 0.13"
+        rpy="0 0 0" />
+      <geometry>
+    <cylinder length="0.3" radius="0.25"/>
+    </geometry>
     </collision>
   </link>
@@ -288,10 +285,9 @@
     <collision>
       <origin
-        xyz="0 0 0"
-        rpy="0 0 0" />
-      <geometry>
-        <mesh
-          filename="package://dql_robot/meshes_object_disposer_robot/right_front.STL" />
-      </geometry>
+        xyz="0 0 0.13"
+        rpy="0 pi 0" />
+      <geometry>
+    <cylinder length="0.3" radius="0.12"/>
+    </geometry>
     </collision>
   </link>
@@ -341,10 +337,9 @@
     <collision>
       <origin
-        xyz="0 0 0"
-        rpy="0 0 0" />
-      <geometry>
-        <mesh
-          filename="package://dql_robot/meshes_object_disposer_robot/right_front_r.STL" />
-      </geometry>
+        xyz="0 0 -0.13"
+        rpy="0 0 0" />
+      <geometry>
+    <cylinder length="0.3" radius="0.25"/>
+    </geometry>
     </collision>
   </link>
@@ -394,10 +389,9 @@
     <collision>
       <origin
-        xyz="0 0 0"
-        rpy="0 0 0" />
-      <geometry>
-        <mesh
-          filename="package://dql_robot/meshes_object_disposer_robot/right_back.STL" />
-      </geometry>
+        xyz="0 0 -0.13"
+        rpy="0 pi 0" />
+      <geometry>
+    <cylinder length="0.3" radius="0.12"/>
+    </geometry>
     </collision>
   </link>
@@ -447,10 +441,9 @@
     <collision>
       <origin
-        xyz="0 0 0"
-        rpy="0 0 0" />
-      <geometry>
-        <mesh
-          filename="package://dql_robot/meshes_object_disposer_robot/right_back_r.STL" />
-      </geometry>
+        xyz="0 0 -0.13"
+        rpy="0 0 0" />
+      <geometry>
+    <cylinder length="0.3" radius="0.25"/>
+    </geometry>
     </collision>
   </link>

Commit message: 11.12.19

File: dql_robot/urdf/object_disposer_robot/my_robot_a.SLDASM.urdf.xacro (robot description, xacro)
@@ -557,5 +557,5 @@
   <joint name="camera_joint2" type="fixed">
     <axis xyz="0 -1 0" />
-    <origin xyz="-20.0 0.0 12.0" rpy="0 1.545 3.14"/>
+    <origin xyz="-20.0 0.0 14.0" rpy="0 1.545 3.14"/>
     <parent link="base_link"/>
     <child link="camera_link2"/>

Commit message: 15.12.19

File: dql_robot/urdf/object_disposer_robot/my_robot_a.SLDASM.urdf.xacro (robot description, xacro)
@@ -557,5 +557,5 @@
   <joint name="camera_joint2" type="fixed">
     <axis xyz="0 -1 0" />
-    <origin xyz="-20.0 0.0 14.0" rpy="0 1.545 3.14"/>
+    <origin xyz="-16.0 0.0 15.0" rpy="0 1.545 3.14"/>
     <parent link="base_link"/>
     <child link="camera_link2"/>

Commit message: 22.12.19

File: dql_robot/urdf/object_disposer_robot/my_robot_a.SLDASM.urdf.xacro (robot description, xacro)
@@ -557,5 +557,5 @@
   <joint name="camera_joint2" type="fixed">
     <axis xyz="0 -1 0" />
-    <origin xyz="-16.0 0.0 15.0" rpy="0 1.545 3.14"/>
+    <origin xyz="-10.0 0.0 12.0" rpy="0 1.545 3.14"/>
     <parent link="base_link"/>
     <child link="camera_link2"/>
@@ -565,5 +565,5 @@
       <update_rate>30.0</update_rate>
       <camera name="head">
-        <horizontal_fov>1.3</horizontal_fov>
+        <horizontal_fov>1.6</horizontal_fov>
         <image>
           <width>640</width>

Commit message: before laser

File: dql_robot/urdf/object_disposer_robot/my_robot_a.SLDASM.urdf.xacro (robot description, xacro)
@@ -80,5 +80,5 @@
         rpy="0 pi 0" />
       <geometry>
-    <cylinder length="0.3" radius="0.12"/>
+    <cylinder length="0.1" radius="0.25"/>
     </geometry>
     </collision>
@@ -97,6 +97,5 @@
       xyz="0 1 0" />
   </joint>
-  <link
-    name="left_front_r">
+  <link name="left_front_r">
     <inertial>
       <origin
@@ -132,5 +131,5 @@
         rpy="0 0 0" />
       <geometry>
-    <cylinder length="0.3" radius="0.25"/>
+    <cylinder length="0.1" radius="0.25"/>
     </geometry>
     </collision>
@@ -184,5 +183,5 @@
         rpy="0 pi 0" />
       <geometry>
-    <cylinder length="0.3" radius="0.12"/>
+        <cylinder length="0.1" radius="0.25"/>
     </geometry>
     </collision>
@@ -236,5 +235,5 @@
         rpy="0 0 0" />
       <geometry>
-    <cylinder length="0.3" radius="0.25"/>
+    <cylinder length="0.1" radius="0.25"/>
     </geometry>
     </collision>
@@ -288,5 +287,5 @@
         rpy="0 pi 0" />
       <geometry>
-    <cylinder length="0.3" radius="0.12"/>
+        <cylinder length="0.1" radius="0.25"/>
     </geometry>
     </collision>
@@ -340,5 +339,5 @@
         rpy="0 0 0" />
       <geometry>
-    <cylinder length="0.3" radius="0.25"/>
+    <cylinder length="0.1" radius="0.25"/>
     </geometry>
     </collision>
@@ -392,5 +391,5 @@
         rpy="0 pi 0" />
       <geometry>
-    <cylinder length="0.3" radius="0.12"/>
+        <cylinder length="0.1" radius="0.25"/>
     </geometry>
     </collision>
@@ -441,8 +440,8 @@
     <collision>
       <origin
-        xyz="0 0 -0.13"
-        rpy="0 0 0" />
-      <geometry>
-    <cylinder length="0.3" radius="0.25"/>
+        xyz="0 -0.011 -0.13"
+        rpy="0 0 0" />
+      <geometry>
+    <cylinder length="0.1" radius="0.25"/>
     </geometry>
     </collision>
@@ -488,12 +487,23 @@
     <material>Gazebo/ZincYellow  </material>
   </gazebo>
-<gazebo reference="lf"/>
-<gazebo reference="rf"/>
-<gazebo reference="lb"/>
-<gazebo reference="rv"/>
+<gazebo reference="lf">
+  <mu1>1.7</mu1>
+  <mu2>0.7</mu2>
+</gazebo>
+<gazebo reference="rf">
+  <mu1>1.7</mu1>
+  <mu2>0.7</mu2>
+</gazebo>
+<gazebo reference="lb">
+  <mu1>1.7</mu1>
+  <mu2>0.7</mu2>
+</gazebo>
+<gazebo reference="rv">
+  <mu1>1.7</mu1>
+  <mu2>0.7</mu2>
+</gazebo>
 <gazebo>
   <plugin name="skid_steer_drive_controller" filename="libgazebo_ros_skid_steer_drive.so">
-    <updateRate>100.0</updateRate>
-    <!--<robotNamespace>/</robotNamespace>-->
+    <updateRate>50.0</updateRate>
     <leftFrontJoint>lf</leftFrontJoint>
     <rightFrontJoint>rf</rightFrontJoint>
@@ -641,5 +651,5 @@
    <joint name="hokuyo_joint" type="fixed">
     <axis xyz="0 1 0" />
-    <origin xyz="-1.1 0 0.20" rpy="0 0 3.1415"/>
+    <origin xyz="-1.2 0 0.25" rpy="0 0 3.1415"/>
     <parent link="base_link"/>
     <child link="hokuyo_link"/>
@@ -669,5 +679,5 @@
    <sensor type="ray" name="head_hokuyo_sensor">
       <pose>0 0 0 0 0 0</pose>
-      <visualize>true</visualize>
+      <visualize>False</visualize>
       <update_rate>100</update_rate>
       <ray>
@@ -682,5 +692,5 @@
         <range>
           <min>0.1</min>
-          <max>50.0</max>
+          <max>52.0</max>
           <resolution>0.1</resolution>
         </range>

Commit message: new dqn

File: dql_robot/urdf/object_disposer_robot/my_robot_a.SLDASM.urdf.xacro (robot description, xacro)
@@ -576,5 +576,5 @@
   <joint name="camera_joint2" type="fixed">
     <axis xyz="0 -1 0" />
-    <origin xyz="-10.0 0.0 9.5" rpy="0 1.545 3.14"/> <!--z=12-->
+    <origin xyz="0 0.0 4.5" rpy="0 1.545 3.14"/> <!--z=9.5 x=-10-->
     <parent link="base_link"/>
     <child link="camera_link2"/>
